File: Launchpad.sch (KiCad schematic (older format))
At the start: 10 parts

Commit message: Blockschaltbild komplett v1
Connections:
- net ~RST: now reaches U?.16 (~RST)
- no-connect marks 1 -> 0
Changed lines of the file:
@@
 $Descr A4 11693 8268
 encoding utf-8
-Sheet 6 6
+Sheet 6 10
 Title ""
 Date ""
@@
 	-1   0    0    -1
 $EndComp
-NoConn ~ 5350 5300
 $Comp
 L power:GND #PWR?
@@
 Wire Wire Line
 	1950 2650 1950 2900
+Text HLabel 5550 5300 2    50   Output ~ 0
+~RST
+Wire Wire Line
+	5550 5300 5350 5300
 $EndSCHEMATC

Commit message: Erste fertige Version
Parts:
- added C? (x2): 4µ7, symbol Device:C_Small
- added D?: LED_Small, symbol Device:LED_Small
- added D?: D_Schottky_Small, symbol Device:D_Schottky_Small
- added J?: USB_OTG, symbol Connector:USB_OTG
- added J?: Conn_01x04_Male, symbol Connector:Conn_01x04_Male
- added J?: Conn_01x04_Female, symbol Connector:Conn_01x04_Female
- added JP? (x4): JP_3, symbol Jumper:Jumper_3_Bridged12
- added JP?: Jumper, symbol Device:Jumper
- added R?: 2k2, symbol Device:R_Small
- added R?: 220, symbol Device:R_Small
- added U?: MCP73831, Package_TO_SOT_SMD:SOT-23-5, symbol Battery_Management:MCP73831-2-OT
Connections:
- net +5V: now also JP?.2
- net GND: now also C?.2, C?.2, J?.4 (Pin_4), R?.2, U?.2 (VSS)
- net VBUS: now also C?.1, D?.1 (K), D?.2 (A), J?.1 (Pin_1), JP?.1, U?.4 (VDD)
- net at J?.2 (D-): now also J?.2 (Pin_2)
- net at J?.3 (D+): now also J?.3 (Pin_3)
- net P1.2: no longer names the net of U?.35 (P1.2)
- net P1.2: now also JP?.2 (C)
- net P1.3: no longer names the net of U?.36 (P1.3)
- net P1.3: now also JP?.2 (C)
- net P1.4: no longer names the net of U?.37 (P1.4)
- net P1.4: now also JP?.2 (C)
- net P1.5: no longer names the net of U?.38 (P1.5)
- net P1.5: now also JP?.2 (C)
- new net: J?.1 (Pin_1), J?.1 (VBUS)
- new net: J?.2 (D-), J?.2 (Pin_2)
- new net: J?.3 (D+), J?.3 (Pin_3)
- new net: J?.4 (ID), J?.4 (Pin_4), J?.5 (GND)
- new net: R?.2, U?.1 (STAT)
- new net: R?.1, U?.5 (PROG)
- new net: D?.1 (K), R?.1
- new net +BATT: C?.1, D?.2 (A), U?.3 (VBAT)
- new net P1.2_LED: JP?.1 (A)
- new net P1.2_XBEE: JP?.3 (B)
- new net P1.3_LED: JP?.1 (A)
- new net P1.3_XBEE: JP?.3 (B)
- new net P1.4_LED: JP?.1 (A)
- new net P1.4_XBEE: JP?.3 (B)
- new net P1.5_FAN: JP?.1 (A)
- new net P1.5_XBEE: JP?.3 (B)
- no-connect marks 0 -> 1
Other:
- note added: "USB-Verbindung entweder über die Basisplatine mit einem breakout-Board als "Kabelersatz" \noder direkt am Launchpad, dann muss der Jumper zw. VBUS und 5V gesteckt werden"
- moved on the sheet: C?, U?, U?A, U?B, U?C, U?D
