File: Launchpad.sch (KiCad schematic (older format))
At the start: 33 parts

Commit message: da war noch nicht alles gespeichert
Parts:
- added R?: 10k, symbol Device:R_Small
Connections:
- wire segments 126 -> 128
Changed lines of the file:
@@
 Wire Wire Line
 	1350 4900 4200 4900
+$Comp
+L Device:R_Small R?
+U 1 1 5F4F4CA4
+P 9400 2850
+F 0 "R?" H 9459 2896 50  0000 L CNN
+F 1 "10k" H 9459 2805 50  0000 L CNN
+F 2 "" H 9400 2850 50  0001 C CNN
+F 3 "~" H 9400 2850 50  0001 C CNN
+	1    9400 2850
+	1    0    0    -1
+$EndComp
+$Comp
+L power:GND #PWR?
+U 1 1 5F4F53E0
+P 9400 3400
+F 0 "#PWR?" H 9400 3150 50  0001 C CNN
+F 1 "GND" H 9405 3227 50  0000 C CNN
+F 2 "" H 9400 3400 50  0001 C CNN
+F 3 "" H 9400 3400 50  0001 C CNN
+	1    9400 3400
+	1    0    0    -1
+$EndComp
+Wire Wire Line
+	9400 3400 9400 2950
+Wire Wire Line
+	9400 2750 9400 2150
 $EndSCHEMATC

Commit message: Bauteile grob platziert
Parts:
- removed C?: 10µ, symbol Device:C_Small
- removed J?: USB_OTG, symbol Connector:USB_OTG
- removed J?: USB_B, symbol Connector:USB_B
- removed J?: Conn_01x04_Male, symbol Connector:Conn_01x04_Male
- removed J?: Conn_01x04_Female, symbol Connector:Conn_01x04_Female
- removed JP?: Jumper, symbol Device:Jumper
- removed R?: 1meg, symbol Device:R_Small
- removed SW?: SW_SPST, symbol Switch:SW_SPST
- added SW3: SW_SPDT, HS-Wismar:SS_13PLP, symbol Switch:SW_SPDT
- C18, C19, C20, C21: renamed from C?; footprint (none) -> Capacitor_SMD:C_1206_3216Metric_Pad1.42x1.75mm_HandSolder
- C22, C23: renamed from C?; footprint (none) -> Capacitor_SMD:C_0603_1608Metric_Pad1.05x0.95mm_HandSolder
- D15: renamed from D?; footprint (none) -> LED_SMD:LED_0603_1608Metric
- J18: renamed from J?; footprint (none) -> TerminalBlock_Phoenix:TerminalBlock_Phoenix_MKDS-3-2-5.08_1x02_P5.08mm_Horizontal
- JP1, JP3, JP4, JP5: renamed from JP?; footprint (none) -> Connector_PinHeader_2.54mm:PinHeader_1x03_P2.54mm_Vertical
- R49, R50, R51, R52, R53: renamed from R?; footprint (none) -> Resistor_SMD:R_0603_1608Metric_Pad1.05x0.95mm_HandSolder
- U10: renamed from U?; footprint (none) -> HS-Wismar:TI_Launchpad
- U12: renamed from U?; footprint (none) -> Package_TO_SOT_SMD:SOT-223-6
- gave numbers to parts that had none: 4
Connections:
- net labels removed: +5V, VDC
- wire segments 128 -> 102
Other:
- note added: "Der 3V3 Jumper auf dem Launchpad muss gezogen sein"
- note removed: "USB-Verbindung entweder über die Basisplatine mit einem breakout-Board als "Kabelersatz" \noder direkt am Launchpad, dann muss der Jumper zw. VBUS und 5V gesteckt werden.\nDer 3V3 Jumper auf dem Launchpad muss gezogen sein"
- moved on the sheet: C18, C19, C20, C21, C22, C23, D15, R49, R50, R51, R52, R53

Commit message: Alle Bauteile platziert
Alle Bauteile sind grob plaziert.
Einige Bauteile sollten noch umplaziert werden (u. a. die Jumper links neben Groov-Con, RGB-LED,).
Parts:
- C18, C19, C20, C21, C22, C23: symbol Device:C_Small -> MCT_Labor_5529-rescue:C_Small-Device
- D14, D16: symbol Diode:BAT54C -> MCT_Labor_5529-rescue:BAT54C-Diode
- D15: symbol Device:LED_Small -> MCT_Labor_5529-rescue:LED_Small-Device
- J18: symbol Connector:Screw_Terminal_01x02 -> MCT_Labor_5529-rescue:Screw_Terminal_01x02-Connector
- JP1, JP3, JP4, JP5: symbol Jumper:Jumper_3_Bridged12 -> MCT_Labor_5529-rescue:Jumper_3_Bridged12-Jumper
- Q1: symbol Transistor_FET:BSS138 -> MCT_Labor_5529-rescue:BSS138-Transistor_FET
- R49, R50, R51, R52, R53: symbol Device:R_Small -> MCT_Labor_5529-rescue:R_Small-Device
- SW3: symbol Switch:SW_SPDT -> MCT_Labor_5529-rescue:SW_SPDT-Switch
- U10: symbol HS-Wismar:msp-exp430f5529-LP -> MCT_Labor_5529-rescue:msp-exp430f5529-LP-HS-Wismar
- U11: symbol Battery_Management:MCP73831-2-OT -> MCT_Labor_5529-rescue:MCP73831-2-OT-Battery_Management
- U12: symbol HS-Wismar:TPS737xx -> MCT_Labor_5529-rescue:TPS737xx-HS-Wismar
Changed lines of the file:
@@
 $EndDescr
 $Comp
-L HS-Wismar:msp-exp430f5529-LP U?
+L MCT_Labor_5529-rescue:msp-exp430f5529-LP-HS-Wismar U?
 U 1 1 5F0CDEE6
 P 3600 5950
@@
 $EndComp
 $Comp
-L HS-Wismar:msp-exp430f5529-LP U?
+L MCT_Labor_5529-rescue:msp-exp430f5529-LP-HS-Wismar U?
 U 2 1 5F0CDEEC
 P 7250 5950
@@
 $EndComp
 $Comp
-L HS-Wismar:msp-exp430f5529-LP U?
+L MCT_Labor_5529-rescue:msp-exp430f5529-LP-HS-Wismar U?
 U 3 1 5F0CDEF2
 P 3850 5950
@@
 $EndComp
 $Comp
-L HS-Wismar:msp-exp430f5529-LP U?
+L MCT_Labor_5529-rescue:msp-exp430f5529-LP-HS-Wismar U?
 U 4 1 5F0CDEF8
 P 6950 5950
@@
 $EndComp
 $Comp
-L power:GND #PWR?
+L MCT_Labor_5529-rescue:GND-power #PWR?
 U 1 1 5F0CDF19
 P 4300 6100
@@
 $EndComp
 $Comp
-L power:GND #PWR?
+L MCT_Labor_5529-rescue:GND-power #PWR?
 U 1 1 5F0CDF1F
 P 7700 6100
@@
 P8.1
 $Comp
-L power:GND #PWR?
+L MCT_Labor_5529-rescue:GND-power #PWR?
 U 1 1 5F0EC63B
 P 7200 3050
@@
 	7200 3050 7200 2050
 $Comp
-L power:+3.3V #PWR0211
+L MCT_Labor_5529-rescue:+3.3V-power #PWR0211
 U 1 1 5F0F48F8
 P 7850 1350
@@
 	7850 1350 7850 1700
 $Comp
-L Device:C_Small C21
+L MCT_Labor_5529-rescue:C_Small-Device C21
 U 1 1 5F0F633F
 P 6350 2500
@@
 Connection ~ 7850 1700
 $Comp
-L power:GND #PWR?
+L MCT_Labor_5529-rescue:GND-power #PWR?
 U 1 1 5F0FA0A5
 P 6350 3050
@@
 $EndComp
 $Comp
-L power:GND #PWR?
+L MCT_Labor_5529-rescue:GND-power #PWR?
 U 1 1 5F0FB479
 P 7850 3050
@@
 P1.5_FAN
 $Comp
-L Jumper:Jumper_3_Bridged12 JP5
+L MCT_Labor_5529-rescue:Jumper_3_Bridged12-Jumper JP5
 U 1 1 5F00A1A8
 P 6150 4000
@@
 P1.5_XBEE
 $Comp
-L power:+BATT #PWR0219
+L MCT_Labor_5529-rescue:+BATT-power #PWR0219
 U 1 1 5F177C72
 P 6050 1350
@@
 P1.2_XBEE
 $Comp
-L Jumper:Jumper_3_Bridged12 JP4
+L MCT_Labor_5529-rescue:Jumper_3_Bridged12-Jumper JP4
 U 1 1 5F01B518
 P 5850 4200
@@
 $EndComp
 $Comp
-L Jumper:Jumper_3_Bridged12 JP3
+L MCT_Labor_5529-rescue:Jumper_3_Bridged12-Jumper JP3
 U 1 1 5F019EE6
 P 5550 4400
@@
 $EndComp
 $Comp
-L Jumper:Jumper_3_Bridged12 JP1
+L MCT_Labor_5529-rescue:Jumper_3_Bridged12-Jumper JP1
 U 1 1 5F0146F8
 P 5250 4600
@@
 	6150 5200 6600 5200
 $Comp
-L power:+3.3V #PWR0223
+L MCT_Labor_5529-rescue:+3.3V-power #PWR0223
 U 1 1 5F01BECD
 P 3150 3850
@@
 	3250 5000 3150 5000
 $Comp
-L power:VCC #PWR0224
+L MCT_Labor_5529-rescue:VCC-power #PWR0224
 U 1 1 5F04B85D
 P 2950 1350
@@
 $EndComp
 $Comp
-L power:GND #PWR0225
+L MCT_Labor_5529-rescue:GND-power #PWR0225
 U 1 1 5F052F05
 P 2950 3050
@@
 $EndComp
 $Comp
-L Connector:Screw_Terminal_01x02 J18
+L MCT_Labor_5529-rescue:Screw_Terminal_01x02-Connector J18
 U 1 1 5F053992
 P 2750 2100
@@
 $EndComp
 $Comp
-L power:GND #PWR?
+L MCT_Labor_5529-rescue:GND-power #PWR?
 U 1 1 5F05E423
 P 3150 3050
@@
 $EndComp
 $Comp
-L Device:C_Small C18
+L MCT_Labor_5529-rescue:C_Small-Device C18
 U 1 1 5F05E429
 P 3150 2150
@@
 $EndComp
 $Comp
-L power:VDD #PWR0227
+L MCT_Labor_5529-rescue:VDD-power #PWR0227
 U 1 1 5F1CD1DC
 P 6800 1350
@@
 $EndComp
 $Comp
-L Diode:BAT54C D16
+L MCT_Labor_5529-rescue:BAT54C-Diode D16
 U 1 1 5F240C6E
 P 6350 1450
@@
 	4700 1550 4700 1800
 $Comp
-L Diode:BAT54C D14
+L MCT_Labor_5529-rescue:BAT54C-Diode D14
 U 1 1 5F246996
 P 4700 1350
@@
 	5750 1350 5750 2600
 $Comp
-L power:VDD #PWR0229
+L MCT_Labor_5529-rescue:VDD-power #PWR0229
 U 1 1 5F2007DF
 P 5750 1350
@@
 	1    0    0    -1
 $EndComp
-$Comp
-L power:VDD #PWR0231
-U 1 1 5F1C2D76
-P 5200 1350
-F 0 "#PWR0231" H 5200 1200 50  0001 C CNN
-F 1 "VDD" H 5215 1523 50  0000 C CNN
-F 2 "" H 5200 1350 50  0001 C CNN
-F 3 "" H 5200 1350 50  0001 C CNN
-	1    5200 1350
-	1    0    0    -1
-$EndComp
 Wire Wire Line
 	3450 3050 3450 3000
 $Comp
-L power:GND #PWR0232
+L MCT_Labor_5529-rescue:GND-power #PWR0232
 U 1 1 5F1ACE91
 P 3450 3050
@@
 Connection ~ 3450 2800
 $Comp
-L power:VBUS #PWR0233
+L MCT_Labor_5529-rescue:VBUS-power #PWR0233
 U 1 1 5F19A070
 P 5000 1350
@@
 	4700 1550 5200 1550
 $Comp
-L Device:R_Small R49
+L MCT_Labor_5529-rescue:R_Small-Device R49
 U 1 1 5F122679
 P 3450 2900
@@
 Connection ~ 4200 2200
 $Comp
-L Transistor_FET:BSS138 Q1
+L MCT_Labor_5529-rescue:BSS138-Transistor_FET Q1
 U 1 1 5F0FF1E3
 P 3650 2800
@@
 	3750 3050 3750 3000
 $Comp
-L power:GND #PWR0234
+L MCT_Labor_5529-rescue:GND-power #PWR0234
 U 1 1 5F0F9E17
 P 3750 3050
@@
 	3750 2400 3750 2200
 $Comp
-L Device:R_Small R50
+L MCT_Labor_5529-rescue:R_Small-Device R50
 U 1 1 5F0E2820
 P 3750 2500
@@
 	5550 3050 5550 2800
 $Comp
-L power:GND #PWR0235
+L MCT_Labor_5529-rescue:GND-power #PWR0235
 U 1 1 5F15FDD6
 P 5550 3050
@@
 $EndComp
 $Comp
-L power:GND #PWR0236
+L MCT_Labor_5529-rescue:GND-power #PWR0236
 U 1 1 5F15F0EF
 P 5750 3050
@@
 	5550 2600 5550 2000
 $Comp
-L Device:C_Small C19
+L MCT_Labor_5529-rescue:C_Small-Device C19
 U 1 1 5F156A80
 P 5750 2700
@@
 $EndComp
 $Comp
-L Device:C_Small C20
+L MCT_Labor_5529-rescue:C_Small-Device C20
 U 1 1 5F15664D
 P 5550 2700
@@
 $EndComp
 $Comp
-L Device:LED_Small D15
+L MCT_Labor_5529-rescue:LED_Small-Device D15
 U 1 1 5F14F51E
 P 5200 1650
@@
 	5200 1950 5200 2200
 $Comp
-L Device:R_Small R52
+L MCT_Labor_5529-rescue:R_Small-Device R52
 U 1 1 5F14006A
 P 5200 1850
@@
 	5550 1350 5550 2000
 $Comp
-L power:+BATT #PWR0237
+L MCT_Labor_5529-rescue:+BATT-power #PWR0237
 U 1 1 5F104E02
 P 5550 1350
@@
 $EndComp
 $Comp
-L power:GND #PWR0238
+L MCT_Labor_5529-rescue:GND-power #PWR0238
 U 1 1 5F1047C0
 P 4700 3050
@@
 $EndComp
 $Comp
-L power:GND #PWR0239
+L MCT_Labor_5529-rescue:GND-power #PWR0239
 U 1 1 5F10418D
 P 4200 3050
@@
 	4200 2600 4200 2200
 $Comp
-L Device:R_Small R51
+L MCT_Labor_5529-rescue:R_Small-Device R51
 U 1 1 5F100A4C
 P 4200 2700
@@
 	1    0    0    -1
 $EndComp
-$Comp
-L Battery_Management:MCP73831-2-OT U11
-U 1 1 5F0DECAC
-P 4700 2100
-F 0 "U11" H 4450 2350 50  0000 C CNN
-F 1 "MCP73831" H 4950 2350 50  0000 C CNN
-F 2 "Package_TO_SOT_SMD:SOT-23-5" H 4750 1850 50  0001 L CIN
-F 3 "http://ww1.microchip.com/downloads/en/DeviceDoc/20001984g.pdf" H 4550 2050 50  0001 C CNN
-	1    4700 2100
-	1    0    0    -1
-$EndComp
 Text Notes 5800 3400 0    50   ~ 0
 Der 3V3 Jumper auf dem Launchpad muss gezogen sein
 $Comp
-L HS-Wismar:TPS737xx U12
+L MCT_Labor_5529-rescue:TPS737xx-HS-Wismar U12
 U 1 1 5F3B50C2
 P 6950 1950
@@
 	6800 1800 6850 1800
 $Comp
-L Device:C_Small C22
+L MCT_Labor_5529-rescue:C_Small-Device C22
 U 1 1 5F3FA9C6
 P 7600 2550
@@
 $EndComp
 $Comp
-L power:GND #PWR?
+L MCT_Labor_5529-rescue:GND-power #PWR?
 U 1 1 5F3FA9CC
 P 7600 3050
@@
 	7600 1800 7600 2450
 $Comp
-L Device:C_Small C23
+L MCT_Labor_5529-rescue:C_Small-Device C23
 U 1 1 5F4041DB
 P 7850 2550
@@
 	3050 4000 5900 4000
 $Comp
-L Device:R_Small R53
+L MCT_Labor_5529-rescue:R_Small-Device R53
 U 1 1 5F4F4CA4
 P 6800 2500
@@
 $EndComp
 $Comp
-L power:GND #PWR0241
+L MCT_Labor_5529-rescue:GND-power #PWR0241
 U 1 1 5F4F53E0
 P 6800 3050
@@
 	6800 2400 6800 1800
 $Comp
-L Switch:SW_SPDT SW3
+L MCT_Labor_5529-rescue:SW_SPDT-Switch SW3
 U 1 1 5F0D41F8
 P 6550 1900
@@
 	6750 1800 6800 1800
 $Comp
-L power:VBUS #PWR0209
+L MCT_Labor_5529-rescue:VBUS-power #PWR0209
 U 1 1 5F168369
 P 4300 3850
@@
 $EndComp
 $Comp
-L power:VCC #PWR0214
+L MCT_Labor_5529-rescue:VCC-power #PWR0214
 U 1 1 5F1A1AD0
 P 3450 1350
@@
 Connection ~ 3450 1350
 $Comp
-L power:VCC #PWR0215
+L MCT_Labor_5529-rescue:VCC-power #PWR0215
 U 1 1 5F1E7553
 P 3150 1350
@@
 Wire Wire Line
 	3150 2250 3150 3050
+$Comp
+L MCT_Labor_5529-rescue:MCP73831-2-OT-Battery_Management U11
+U 1 1 5F0DECAC
+P 4700 2100
+F 0 "U11" H 4450 2350 50  0000 C CNN
+F 1 "MCP73831" H 4950 2350 50  0000 C CNN
+F 2 "Package_TO_SOT_SMD:SOT-23-5" H 4750 1850 50  0001 L CIN
+F 3 "http://ww1.microchip.com/downloads/en/DeviceDoc/20001984g.pdf" H 4550 2050 50  0001 C CNN
+	1    4700 2100
+	1    0    0    -1
+$EndComp
+$Comp
+L MCT_Labor_5529-rescue:VDD-power #PWR0231
+U 1 1 5F1C2D76
+P 5200 1350
+F 0 "#PWR0231" H 5200 1200 50  0001 C CNN
+F 1 "VDD" H 5215 1523 50  0000 C CNN
+F 2 "" H 5200 1350 50  0001 C CNN
+F 3 "" H 5200 1350 50  0001 C CNN
+	1    5200 1350
+	1    0    0    -1
+$EndComp
 $EndSCHEMATC
