File: Launchpad.sch (KiCad schematic (older format))
At the start: 31 parts, among them J18 Screw_Terminal_01x02, Q1 BSS138, SW3 SW_SPDT, U10 msp-exp430f5529-LP, U11 MCP73831, U12 TPS73733, U13 TLV61048

Commit message: minor glitches
Parts:
- R54: value 107k -> 100k
Connections:
- net VCC renamed VDC
- net ~RST: no longer names the net of U10.16 (~RST)
- no-connect marks 0 -> 1
Other:
- moved on the sheet: C17, C21, D16, SW3
Changed lines of the file:
@@
 L MCT_Labor_5529-rescue:C_Small-Device C21
 U 1 1 5F0F633F
-P 6350 2500
-F 0 "C21" H 6442 2546 50  0000 L CNN
-F 1 "10µ" H 6442 2455 50  0000 L CNN
-F 2 "Capacitor_SMD:C_1206_3216Metric_Pad1.42x1.75mm_HandSolder" H 6350 2500 50  0001 C CNN
-F 3 "~" H 6350 2500 50  0001 C CNN
-	1    6350 2500
+P 6250 2500
+F 0 "C21" H 6342 2546 50  0000 L CNN
+F 1 "10µ" H 6342 2455 50  0000 L CNN
+F 2 "Capacitor_SMD:C_1206_3216Metric_Pad1.42x1.75mm_HandSolder" H 6250 2500 50  0001 C CNN
+F 3 "~" H 6250 2500 50  0001 C CNN
+	1    6250 2500
 	1    0    0    -1
 $EndComp
@@
 L MCT_Labor_5529-rescue:GND-power #PWR?
 U 1 1 5F0FA0A5
-P 6350 3050
+P 6250 3050
 AR Path="/5F0FA0A5" Ref="#PWR?"  Part="1"
 AR Path="/5F0B42CA/5F0FA0A5" Ref="#PWR0212"  Part="1"
-F 0 "#PWR0212" H 6350 2800 50  0001 C CNN
-F 1 "GND" H 6355 2877 50  0000 C CNN
-F 2 "" H 6350 3050 50  0001 C CNN
-F 3 "" H 6350 3050 50  0001 C CNN
-	1    6350 3050
+F 0 "#PWR0212" H 6250 2800 50  0001 C CNN
+F 1 "GND" H 6255 2877 50  0000 C CNN
+F 2 "" H 6250 3050 50  0001 C CNN
+F 3 "" H 6250 3050 50  0001 C CNN
+	1    6250 3050
 	1    0    0    -1
 $EndComp
@@
 $EndComp
 Wire Wire Line
-	6350 2600 6350 3050
+	6250 2600 6250 3050
 Wire Wire Line
 	7850 3050 7850 2650
-Text HLabel 7800 5400 2    50   Output ~ 0
-~RST
-Wire Wire Line
-	7800 5400 7600 5400
 Wire Wire Line
 	6600 5300 5850 5300
@@
 L MCT_Labor_5529-rescue:+BATT-power #PWR0219
 U 1 1 5F177C72
-P 6050 1350
-F 0 "#PWR0219" H 6050 1200 50  0001 C CNN
-F 1 "+BATT" H 6065 1523 50  0000 C CNN
-F 2 "" H 6050 1350 50  0001 C CNN
-F 3 "" H 6050 1350 50  0001 C CNN
-	1    6050 1350
+P 5950 1350
+F 0 "#PWR0219" H 5950 1200 50  0001 C CNN
+F 1 "+BATT" H 5965 1523 50  0000 C CNN
+F 2 "" H 5950 1350 50  0001 C CNN
+F 3 "" H 5950 1350 50  0001 C CNN
+	1    5950 1350
 	1    0    0    -1
 $EndComp
@@
 Wire Wire Line
 	3250 5000 3150 5000
-$Comp
-L MCT_Labor_5529-rescue:VCC-power #PWR0224
-U 1 1 5F04B85D
-P 2950 1350
-F 0 "#PWR0224" H 2950 1200 50  0001 C CNN
-F 1 "VCC" H 2965 1523 50  0000 C CNN
-F 2 "" H 2950 1350 50  0001 C CNN
-F 3 "" H 2950 1350 50  0001 C CNN
-	1    2950 1350
-	1    0    0    -1
-$EndComp
 $Comp
 L MCT_Labor_5529-rescue:GND-power #PWR0225
@@
 L MCT_Labor_5529-rescue:BAT54C-Diode D16
 U 1 1 5F240C6E
-P 6350 1450
-F 0 "D16" V 6350 1537 50  0000 L CNN
-F 1 "BAT54C" V 6305 1538 50  0001 L CNN
-F 2 "Package_TO_SOT_SMD:SOT-23" H 6425 1575 50  0001 L CNN
-F 3 "http://www.diodes.com/_files/datasheets/ds11005.pdf" H 6270 1450 50  0001 C CNN
-	1    6350 1450
-	1    0    0    -1
-$EndComp
-Wire Wire Line
-	6050 1350 6050 1450
-Wire Wire Line
-	6350 1650 6350 1700
-Connection ~ 6350 1700
+P 6250 1450
+F 0 "D16" V 6250 1537 50  0000 L CNN
+F 1 "BAT54C" V 6205 1538 50  0001 L CNN
+F 2 "Package_TO_SOT_SMD:SOT-23" H 6325 1575 50  0001 L CNN
+F 3 "http://www.diodes.com/_files/datasheets/ds11005.pdf" H 6170 1450 50  0001 C CNN
+	1    6250 1450
+	1    0    0    -1
+$EndComp
+Wire Wire Line
+	5950 1350 5950 1450
+Wire Wire Line
+	6250 1650 6250 1700
+Connection ~ 6250 1700
 Wire Wire Line
 	2950 3050 2950 2200
 Wire Wire Line
 	2950 2100 2950 1350
-Wire Wire Line
-	3450 1350 4400 1350
 Wire Wire Line
 	3450 1350 3450 2800
@@
 	1    0    0    -1
 $EndComp
-Wire Wire Line
-	6350 1700 6850 1700
 Wire Wire Line
 	7550 1700 7850 1700
@@
 	6800 1350 6800 1450
 Connection ~ 6800 1800
-Wire Wire Line
-	6650 1450 6800 1450
 Connection ~ 6800 1450
 Wire Wire Line
@@
 L MCT_Labor_5529-rescue:SW_SPDT-Switch SW3
 U 1 1 5F0D41F8
-P 6550 1900
-F 0 "SW3" H 6550 1700 50  0000 C CNN
-F 1 "SW_SPDT" H 6550 2094 50  0001 C CNN
-F 2 "HS-Wismar:SS_13PLP" H 6550 1900 50  0001 C CNN
-F 3 "~" H 6550 1900 50  0001 C CNN
-	1    6550 1900
-	1    0    0    -1
-$EndComp
-Wire Wire Line
-	6350 1700 6350 1900
-Connection ~ 6350 1900
-Wire Wire Line
-	6750 1800 6800 1800
+P 6450 1900
+F 0 "SW3" H 6350 2000 50  0000 C CNN
+F 1 "SW_SPDT" H 6450 2094 50  0001 C CNN
+F 2 "HS-Wismar:SS_13PLP" H 6450 1900 50  0001 C CNN
+F 3 "~" H 6450 1900 50  0001 C CNN
+	1    6450 1900
+	1    0    0    -1
+$EndComp
+Wire Wire Line
+	6250 1700 6250 1900
+Connection ~ 6250 1900
 $Comp
 L MCT_Labor_5529-rescue:VBUS-power #PWR0209
@@
 	1    0    0    -1
 $EndComp
-$Comp
-L MCT_Labor_5529-rescue:VCC-power #PWR0214
-U 1 1 5F1A1AD0
-P 3450 1350
-F 0 "#PWR0214" H 3450 1200 50  0001 C CNN
-F 1 "VCC" H 3465 1523 50  0000 C CNN
-F 2 "" H 3450 1350 50  0001 C CNN
-F 3 "" H 3450 1350 50  0001 C CNN
-	1    3450 1350
-	1    0    0    -1
-$EndComp
-Connection ~ 3450 1350
-$Comp
-L MCT_Labor_5529-rescue:VCC-power #PWR0215
-U 1 1 5F1E7553
-P 3150 1350
-F 0 "#PWR0215" H 3150 1200 50  0001 C CNN
-F 1 "VCC" H 3165 1523 50  0000 C CNN
-F 2 "" H 3150 1350 50  0001 C CNN
-F 3 "" H 3150 1350 50  0001 C CNN
-	1    3150 1350
-	1    0    0    -1
-$EndComp
 Wire Wire Line
 	3150 2050 3150 1350
@@
 P 10400 2600
 F 0 "R54" H 10470 2646 50  0000 L CNN
-F 1 "107k" H 10470 2555 50  0000 L CNN
+F 1 "100k" H 10470 2555 50  0000 L CNN
 F 2 "Resistor_SMD:R_0603_1608Metric_Pad1.05x0.95mm_HandSolder" V 10330 2600 50  0001 C CNN
 F 3 "~" H 10400 2600 50  0001 C CNN
@@
 	10200 1850 10400 1850
 Wire Wire Line
-	11000 1850 11000 1700
+	11000 1850 11000 1350
 Connection ~ 10800 1850
 Wire Wire Line
@@
 L power:GND #PWR05
 U 1 1 5F2393ED
-P 10800 2500
-F 0 "#PWR05" H 10800 2250 50  0001 C CNN
-F 1 "GND" H 10805 2327 50  0000 C CNN
-F 2 "" H 10800 2500 50  0001 C CNN
-F 3 "" H 10800 2500 50  0001 C CNN
-	1    10800 2500
+P 10800 3050
+F 0 "#PWR05" H 10800 2800 50  0001 C CNN
+F 1 "GND" H 10805 2877 50  0000 C CNN
+F 2 "" H 10800 3050 50  0001 C CNN
+F 3 "" H 10800 3050 50  0001 C CNN
+	1    10800 3050
 	1    0    0    -1
 $EndComp
@@
 L power:GND #PWR04
 U 1 1 5F239D9A
-P 10400 2900
-F 0 "#PWR04" H 10400 2650 50  0001 C CNN
-F 1 "GND" H 10405 2727 50  0000 C CNN
-F 2 "" H 10400 2900 50  0001 C CNN
-F 3 "" H 10400 2900 50  0001 C CNN
-	1    10400 2900
+P 10400 3050
+F 0 "#PWR04" H 10400 2800 50  0001 C CNN
+F 1 "GND" H 10405 2877 50  0000 C CNN
+F 2 "" H 10400 3050 50  0001 C CNN
+F 3 "" H 10400 3050 50  0001 C CNN
+	1    10400 3050
 	1    0    0    -1
 $EndComp
@@
 L power:GND #PWR03
 U 1 1 5F23AC8B
-P 9450 2650
-F 0 "#PWR03" H 9450 2400 50  0001 C CNN
-F 1 "GND" H 9455 2477 50  0000 C CNN
-F 2 "" H 9450 2650 50  0001 C CNN
-F 3 "" H 9450 2650 50  0001 C CNN
-	1    9450 2650
+P 9450 3050
+F 0 "#PWR03" H 9450 2800 50  0001 C CNN
+F 1 "GND" H 9455 2877 50  0000 C CNN
+F 2 "" H 9450 3050 50  0001 C CNN
+F 3 "" H 9450 3050 50  0001 C CNN
+	1    9450 3050
 	1    0    0    -1
 $EndComp
@@
 L power:GND #PWR02
 U 1 1 5F23B02B
-P 8350 2450
-F 0 "#PWR02" H 8350 2200 50  0001 C CNN
-F 1 "GND" H 8355 2277 50  0000 C CNN
-F 2 "" H 8350 2450 50  0001 C CNN
-F 3 "" H 8350 2450 50  0001 C CNN
-	1    8350 2450
-	1    0    0    -1
-$EndComp
-Wire Wire Line
-	10800 2350 10800 2500
+P 8350 3050
+F 0 "#PWR02" H 8350 2800 50  0001 C CNN
+F 1 "GND" H 8355 2877 50  0000 C CNN
+F 2 "" H 8350 3050 50  0001 C CNN
+F 3 "" H 8350 3050 50  0001 C CNN
+	1    8350 3050
+	1    0    0    -1
+$EndComp
+Wire Wire Line
+	10800 2350 10800 3050
 Wire Wire Line
 	10400 2000 10400 1850
@@
 	10400 2450 10400 2350
 Wire Wire Line
-	10400 2750 10400 2900
+	10400 2750 10400 3050
 Wire Wire Line
 	9750 2350 10400 2350
@@
 Connection ~ 9100 1850
 Wire Wire Line
-	9450 2550 9450 2650
+	9450 2550 9450 3050
 $Comp
 L power:+12V #PWR06
 U 1 1 5F26FEA2
-P 11000 1700
-F 0 "#PWR06" H 11000 1550 50  0001 C CNN
-F 1 "+12V" H 11015 1873 50  0000 C CNN
-F 2 "" H 11000 1700 50  0001 C CNN
-F 3 "" H 11000 1700 50  0001 C CNN
-	1    11000 1700
+P 11000 1350
+F 0 "#PWR06" H 11000 1200 50  0001 C CNN
+F 1 "+12V" H 11015 1523 50  0000 C CNN
+F 2 "" H 11000 1350 50  0001 C CNN
+F 3 "" H 11000 1350 50  0001 C CNN
+	1    11000 1350
 	1    0    0    -1
 $EndComp
@@
 L Device:C C17
 U 1 1 5F20F661
-P 8350 2100
-F 0 "C17" H 8465 2146 50  0000 L CNN
-F 1 "1u" H 8465 2055 50  0000 L CNN
-F 2 "Capacitor_SMD:C_0603_1608Metric_Pad1.05x0.95mm_HandSolder" H 8388 1950 50  0001 C CNN
-F 3 "~" H 8350 2100 50  0001 C CNN
-	1    8350 2100
+P 8350 2550
+F 0 "C17" H 8465 2596 50  0000 L CNN
+F 1 "1u" H 8465 2505 50  0000 L CNN
+F 2 "Capacitor_SMD:C_0603_1608Metric_Pad1.05x0.95mm_HandSolder" H 8388 2400 50  0001 C CNN
+F 3 "~" H 8350 2550 50  0001 C CNN
+	1    8350 2550
 	1    0    0    -1
 $EndComp
@@
 12V_Enable
 Wire Wire Line
-	6350 1900 6350 2100
+	6250 1900 6250 2100
 Wire Wire Line
 	8000 1850 8000 2100
-Wire Wire Line
-	8000 2100 6350 2100
-Connection ~ 6350 2100
-Wire Wire Line
-	6350 2100 6350 2400
+Connection ~ 6250 2100
+Wire Wire Line
+	6250 2100 6250 2400
 Wire Wire Line
 	8000 1850 8350 1850
 Wire Wire Line
-	8350 1850 8350 1950
+	8350 1850 8350 2400
 Connection ~ 8350 1850
 Wire Wire Line
 	8350 1850 9100 1850
 Wire Wire Line
-	8350 2250 8350 2450
+	8350 2700 8350 3050
 Wire Wire Line
 	9100 2350 9150 2350
 Text GLabel 6450 5900 0    50   Input ~ 0
 12V_Enable
+$Comp
+L power:VDC #PWR0102
+U 1 1 5F9B4FE0
+P 2950 1350
+F 0 "#PWR0102" H 2950 1250 50  0001 C CNN
+F 1 "VDC" H 2965 1523 50  0000 C CNN
+F 2 "" H 2950 1350 50  0001 C CNN
+F 3 "" H 2950 1350 50  0001 C CNN
+	1    2950 1350
+	1    0    0    -1
+$EndComp
+$Comp
+L power:VDC #PWR0103
+U 1 1 5F9B6F32
+P 3150 1350
+F 0 "#PWR0103" H 3150 1250 50  0001 C CNN
+F 1 "VDC" H 3165 1523 50  0000 C CNN
+F 2 "" H 3150 1350 50  0001 C CNN
+F 3 "" H 3150 1350 50  0001 C CNN
+	1    3150 1350
+	1    0    0    -1
+$EndComp
+$Comp
+L power:VDC #PWR0104
+U 1 1 5F9BB647
+P 3450 1350
+F 0 "#PWR0104" H 3450 1250 50  0001 C CNN
+F 1 "VDC" H 3465 1523 50  0000 C CNN
+F 2 "" H 3450 1350 50  0001 C CNN
+F 3 "" H 3450 1350 50  0001 C CNN
+	1    3450 1350
+	1    0    0    -1
+$EndComp
+Wire Wire Line
+	6550 1450 6800 1450
+Wire Wire Line
+	6250 1700 6850 1700
+Wire Wire Line
+	6650 1800 6800 1800
+Wire Wire Line
+	6250 2100 8000 2100
+Wire Wire Line
+	3450 1350 4400 1350
+Connection ~ 3450 1350
+NoConn ~ 7600 5400
 $EndSCHEMATC

Commit message: Aktuell gefertigte Variante
Parts:
- C17: value 1u -> 1µ
- C19, C20: value 4µ7 -> 10µ
- C24: value 10u -> 10µ
- D15: footprint LED_SMD:LED_0603_1608Metric -> LED_SMD:LED_0603_1608Metric_Pad1.05x0.95mm_HandSolder
- R48: value 1.5M -> 680k
- R54: value 100k -> 47k
Changed lines of the file:
@@
 P 5750 2700
 F 0 "C19" V 5800 2500 50  0000 L CNN
-F 1 "4µ7" V 5800 2800 50  0000 L CNN
+F 1 "10µ" V 5800 2800 50  0000 L CNN
 F 2 "Capacitor_SMD:C_1206_3216Metric_Pad1.42x1.75mm_HandSolder" H 5750 2700 50  0001 C CNN
 F 3 "~" H 5750 2700 50  0001 C CNN
@@
 P 5550 2700
 F 0 "C20" V 5600 2500 50  0000 L CNN
-F 1 "4µ7" V 5600 2800 50  0000 L CNN
+F 1 "10µ" V 5600 2800 50  0000 L CNN
 F 2 "Capacitor_SMD:C_1206_3216Metric_Pad1.42x1.75mm_HandSolder" H 5550 2700 50  0001 C CNN
 F 3 "~" H 5550 2700 50  0001 C CNN
@@
 F 0 "D15" V 5200 1580 50  0000 R CNN
 F 1 "LED_Small" V 5155 1580 50  0001 R CNN
-F 2 "LED_SMD:LED_0603_1608Metric" V 5200 1650 50  0001 C CNN
+F 2 "LED_SMD:LED_0603_1608Metric_Pad1.05x0.95mm_HandSolder" V 5200 1650 50  0001 C CNN
 F 3 "~" V 5200 1650 50  0001 C CNN
 	1    5200 1650
@@
 P 10400 2150
 F 0 "R48" H 10470 2196 50  0000 L CNN
-F 1 "1.5M" H 10470 2105 50  0000 L CNN
+F 1 "680k" H 10470 2105 50  0000 L CNN
 F 2 "Resistor_SMD:R_0603_1608Metric_Pad1.05x0.95mm_HandSolder" V 10330 2150 50  0001 C CNN
 F 3 "~" H 10400 2150 50  0001 C CNN
@@
 P 10400 2600
 F 0 "R54" H 10470 2646 50  0000 L CNN
-F 1 "100k" H 10470 2555 50  0000 L CNN
+F 1 "47k" H 10470 2555 50  0000 L CNN
 F 2 "Resistor_SMD:R_0603_1608Metric_Pad1.05x0.95mm_HandSolder" V 10330 2600 50  0001 C CNN
 F 3 "~" H 10400 2600 50  0001 C CNN
@@
 P 10800 2200
 F 0 "C24" H 10915 2246 50  0000 L CNN
-F 1 "10u" H 10915 2155 50  0000 L CNN
+F 1 "10µ" H 10915 2155 50  0000 L CNN
 F 2 "Capacitor_SMD:C_1206_3216Metric_Pad1.42x1.75mm_HandSolder" H 10838 2050 50  0001 C CNN
 F 3 "~" H 10800 2200 50  0001 C CNN
@@
 P 8350 2550
 F 0 "C17" H 8465 2596 50  0000 L CNN
-F 1 "1u" H 8465 2505 50  0000 L CNN
+F 1 "1µ" H 8465 2505 50  0000 L CNN
 F 2 "Capacitor_SMD:C_0603_1608Metric_Pad1.05x0.95mm_HandSolder" H 8388 2400 50  0001 C CNN
 F 3 "~" H 8350 2550 50  0001 C CNN
