File: LED-Treiber.sch (KiCad schematic (older format))
At the start: 1 part

Commit message: Bauteile grob platziert
Parts:
- U2: renamed from U?; footprint (none) -> Package_SO:SOIC-16_3.9x9.9mm_P1.27mm
Changed lines of the file:
@@
 $EndDescr
 $Comp
-L Transistor_Array:ULN2003 U?
+L Transistor_Array:ULN2003 U2
 U 1 1 5EF743C0
 P 5400 3600
-F 0 "U?" H 5400 4267 50  0000 C CNN
+F 0 "U2" H 5400 4267 50  0000 C CNN
 F 1 "ULN2003" H 5400 4176 50  0000 C CNN
-F 2 "" H 5450 3050 50  0001 L CNN
+F 2 "Package_SO:SOIC-16_3.9x9.9mm_P1.27mm" H 5450 3050 50  0001 L CNN
 F 3 "http://www.ti.com/lit/ds/symlink/uln2003a.pdf" H 5500 3400 50  0001 C CNN
 	1    5400 3600
@@
 $EndComp
 $Comp
-L power:+5V #PWR?
+L power:+5V #PWR0108
 U 1 1 5EF74EA2
 P 6050 2800
-F 0 "#PWR?" H 6050 2650 50  0001 C CNN
+F 0 "#PWR0108" H 6050 2650 50  0001 C CNN
 F 1 "+5V" H 6065 2973 50  0000 C CNN
 F 2 "" H 6050 2800 50  0001 C CNN
@@
 $EndComp
 $Comp
-L power:GND #PWR?
+L power:GND #PWR0109
 U 1 1 5EF75057
 P 5400 4450
-F 0 "#PWR?" H 5400 4200 50  0001 C CNN
+F 0 "#PWR0109" H 5400 4200 50  0001 C CNN
 F 1 "GND" H 5405 4277 50  0000 C CNN
 F 2 "" H 5400 4450 50  0001 C CNN

Commit message: Alle Bauteile platziert
Alle Bauteile sind grob plaziert.
Einige Bauteile sollten noch umplaziert werden (u. a. die Jumper links neben Groov-Con, RGB-LED,).
Parts:
- U2: symbol Transistor_Array:ULN2003 -> MCT_Labor_5529-rescue:ULN2003-Transistor_Array
Changed lines of the file:
@@
 $EndDescr
 $Comp
-L Transistor_Array:ULN2003 U2
+L MCT_Labor_5529-rescue:ULN2003-Transistor_Array U2
 U 1 1 5EF743C0
 P 5400 3600
@@
 $EndComp
 $Comp
-L power:+5V #PWR0108
+L MCT_Labor_5529-rescue:+5V-power #PWR0108
 U 1 1 5EF74EA2
 P 6050 2800
@@
 $EndComp
 $Comp
-L power:GND #PWR0109
+L MCT_Labor_5529-rescue:GND-power #PWR0109
 U 1 1 5EF75057
 P 5400 4450

Commit message: Anpassungen am Lüfteranschluss und den LEDs
-Lüfteranschluss verändert
 -> 12V-Versorgung eingefügt
-LED & LCD auf 3,3V umgestellt
 -> Ladungspunpe für neg. Kontrastspannung
-keine 5V Versorgung mehr
Connections:
- net labels added: +3.3V
- net labels removed: +5V, LED_7, LED_LCD
Changed lines of the file:
@@
-$EndComp
-$Comp
-L MCT_Labor_5529-rescue:+5V-power #PWR0108
-U 1 1 5EF74EA2
-P 6050 2800
-F 0 "#PWR0108" H 6050 2650 50  0001 C CNN
-F 1 "+5V" H 6065 2973 50  0000 C CNN
-F 2 "" H 6050 2800 50  0001 C CNN
-F 3 "" H 6050 2800 50  0001 C CNN
-	1    6050 2800
-	1    0    0    -1
 $EndComp
 $Comp
@@
 Text HLabel 4750 3900 0    50   Input ~ 0
 LED_6
-Text HLabel 4750 4000 0    50   Input ~ 0
-LED_7
 Wire Wire Line
 	4750 3400 5000 3400
@@
 Text HLabel 6200 3900 2    50   UnSpc ~ 0
 LED_F3
-Text HLabel 6200 4000 2    50   UnSpc ~ 0
-LED_LCD
 Wire Wire Line
 	5800 3400 6200 3400
@@
 Wire Wire Line
 	6200 4000 5800 4000
+$Comp
+L power:+3.3V #PWR015
+U 1 1 5F31B6ED
+P 6050 2800
+F 0 "#PWR015" H 6050 2650 50  0001 C CNN
+F 1 "+3.3V" H 6065 2973 50  0000 C CNN
+F 2 "" H 6050 2800 50  0001 C CNN
+F 3 "" H 6050 2800 50  0001 C CNN
+	1    6050 2800
+	1    0    0    -1
+$EndComp
 $EndSCHEMATC

Commit message: Kleine Anpassungen
Connections:
- wire segments 17 -> 15
Changed lines of the file:
@@
 Wire Wire Line
 	5000 3900 4750 3900
-Wire Wire Line
-	4750 4000 5000 4000
 Text HLabel 6200 3400 2    50   UnSpc ~ 0
 LED_R
@@
 Wire Wire Line
 	5800 3900 6200 3900
-Wire Wire Line
-	6200 4000 5800 4000
 $Comp
 L power:+3.3V #PWR015
