File: SPI.sch (KiCad schematic (older format))
At the start: 7 parts

Commit message: Erste fertige Version
Parts:
- added C? (x2): 100n, symbol Device:C_Small
- added C?: 1µ, symbol Device:C_Small
- added D? (x8): LED_Small, symbol Device:LED_Small
- added J?: Conn_02x05_Odd_Even, symbol Connector_Generic:Conn_02x05_Odd_Even
- added R?: 1meg, symbol Device:R_Small
- added R? (x2): 10k, symbol Device:R_Small
- added R? (x8): 220, symbol Device:R_Small
- added U?: 74HCT595, symbol 74xx:74HCT595
Connections:
- net +3V3: now also C?.1, C?.1, J?.4 (Pin_4), R?.1, U?.16 (VCC)
- net GND: now also C?.2, C?.2, C?.2, J?.8 (Pin_8), R?.1, R?.1, R?.1, R?.1, R?.1, R?.1, R?.1, R?.1, R?.2, R?.2, U?.8 (GND)
- net MISO: now also J?.2 (Pin_2)
- net MOSI: now also J?.10 (Pin_10), U?.14 (SER)
- net SCK: now also J?.6 (Pin_6), U?.11 (SRCLK)
- net at U?.10 (O5): now also J?.5 (Pin_5)
- net at U?.11 (O4): now also J?.3 (Pin_3)
- net at U?.12 (O3): now also J?.1 (Pin_1)
- net at U?.13 (O2): now also U?.12 (RCLK)
- net at U?.7 (O7): now also J?.9 (Pin_9)
- net at U?.9 (O6): now also J?.7 (Pin_7)
- net at J?.11 (SHIELD): now also R?.1
- new net: D?.2 (A), U?.1 (QB)
- new net: C?.1, R?.2, U?.10 (~SRCLR)
- new net: R?.1, U?.13 (~OE)
- new net: D?.2 (A), U?.15 (QA)
- new net: D?.2 (A), U?.2 (QC)
- new net: D?.2 (A), U?.3 (QD)
- new net: D?.2 (A), U?.4 (QE)
- new net: D?.2 (A), U?.5 (QF)
- new net: D?.2 (A), U?.6 (QG)
- new net: D?.2 (A), U?.7 (QH)
- new net: D?.1 (K), R?.2 (x8)
Other:
- moved on the sheet: C?, R?, U?

Commit message: Bauteile grob platziert
Parts:
- C3, C4, C5, C6, C7, C8: renamed from C?; footprint (none) -> Capacitor_SMD:C_0603_1608Metric_Pad1.05x0.95mm_HandSolder
- D2, D3, D4, D5, D6, D7, D8, D9: renamed from D?; footprint (none) -> LED_SMD:LED_0603_1608Metric_Pad1.05x0.95mm_HandSolder
- J1: renamed from J?; footprint (none) -> Connector_Card:microSD_HC_Hirose_DM3D-SF
- J2: renamed from J?; footprint (none) -> Connector_PinHeader_2.54mm:PinHeader_2x05_P2.54mm_Vertical
- R16, R17, R18, R19, R20, R21, R22, R23, R24, R25, R26, R27: renamed from R?; footprint (none) -> Resistor_SMD:R_0603_1608Metric_Pad1.05x0.95mm_HandSolder
- U4, U6: renamed from U?; footprint (none) -> Package_SO:SOIC-16_3.9x9.9mm_P1.27mm
- gave numbers to parts that had none: 1

Commit message: Alle Bauteile platziert
Alle Bauteile sind grob plaziert.
Einige Bauteile sollten noch umplaziert werden (u. a. die Jumper links neben Groov-Con, RGB-LED,).
Parts:
- C3, C4, C5, C6, C7, C8: symbol Device:C_Small -> MCT_Labor_5529-rescue:C_Small-Device
- D2, D3, D4, D5, D6, D7, D8, D9: symbol Device:LED_Small -> MCT_Labor_5529-rescue:LED_Small-Device
- J1: symbol Connector:Micro_SD_Card_Det -> MCT_Labor_5529-rescue:Micro_SD_Card_Det-Connector
- J2: symbol Connector_Generic:Conn_02x05_Odd_Even -> MCT_Labor_5529-rescue:Conn_02x05_Odd_Even-Connector_Generic
- R16, R17, R18, R19, R20, R21, R22, R23, R24, R25, R26, R27: symbol Device:R_Small -> MCT_Labor_5529-rescue:R_Small-Device
- U4: symbol 74xx:74LS138 -> MCT_Labor_5529-rescue:74LS138-74xx
- U5: symbol RF:NRF24L01_Breakout -> MCT_Labor_5529-rescue:NRF24L01_Breakout-RF
- U6: symbol 74xx:74HCT595 -> MCT_Labor_5529-rescue:74HCT595-74xx
Changed lines of the file:
@@
 $EndDescr
 $Comp
-L 74xx:74LS138 U4
+L MCT_Labor_5529-rescue:74LS138-74xx U4
 U 1 1 5EF44FFA
 P 2300 5450
@@
 	1800 5850 1600 5850
 $Comp
-L power:GND #PWR0121
+L MCT_Labor_5529-rescue:GND-power #PWR0121
 U 1 1 5EF477CB
 P 2300 6150
@@
 $EndComp
 $Comp
-L power:GND #PWR0122
+L MCT_Labor_5529-rescue:GND-power #PWR0122
 U 1 1 5EF478AE
 P 1700 6150
@@
 	1700 5750 1800 5750
 $Comp
-L power:+3.3V #PWR0123
+L MCT_Labor_5529-rescue:+3.3V-power #PWR0123
 U 1 1 5EF480CB
 P 2300 4750
@@
 	2300 4750 2300 4850
 $Comp
-L power:+3.3V #PWR0124
+L MCT_Labor_5529-rescue:+3.3V-power #PWR0124
 U 1 1 5EF483EB
 P 1700 4750
@@
 	1700 5650 1800 5650
 $Comp
-L Device:R_Small R16
+L MCT_Labor_5529-rescue:R_Small-Device R16
 U 1 1 5EF49E2C
 P 1600 5650
@@
 	1600 5850 1400 5850
 $Comp
-L power:+3.3V #PWR0125
+L MCT_Labor_5529-rescue:+3.3V-power #PWR0125
 U 1 1 5EF4A54D
 P 1600 4750
@@
 	1600 4750 1600 5550
 $Comp
-L Device:C_Small C3
+L MCT_Labor_5529-rescue:C_Small-Device C3
 U 1 1 5EF4BF4E
 P 950 5550
@@
 $EndComp
 $Comp
-L power:+3.3V #PWR0126
+L MCT_Labor_5529-rescue:+3.3V-power #PWR0126
 U 1 1 5EF4C200
 P 950 4750
@@
 $EndComp
 $Comp
-L power:GND #PWR0127
+L MCT_Labor_5529-rescue:GND-power #PWR0127
 U 1 1 5EF4C7FB
 P 950 6150
@@
 NoConn ~ 3750 2600
 $Comp
-L Device:C_Small C4
+L MCT_Labor_5529-rescue:C_Small-Device C4
 U 1 1 5EF62DE3
 P 2500 3350
@@
 $EndComp
 $Comp
-L power:GND #PWR0128
+L MCT_Labor_5529-rescue:GND-power #PWR0128
 U 1 1 5EF6351E
 P 3550 4100
@@
 	3350 2900 3350 2600
 $Comp
-L power:+3.3V #PWR0129
+L MCT_Labor_5529-rescue:+3.3V-power #PWR0129
 U 1 1 5EF673F0
 P 2500 2150
@@
 Connection ~ 2500 2900
 $Comp
-L power:GND #PWR0130
+L MCT_Labor_5529-rescue:GND-power #PWR0130
 U 1 1 5EF6C589
 P 2500 4100
@@
 	2500 4100 2500 3450
 $Comp
-L RF:NRF24L01_Breakout U5
+L MCT_Labor_5529-rescue:NRF24L01_Breakout-RF U5
 U 1 1 5EF74F9D
 P 6150 1650
@@
 $EndComp
 $Comp
-L Connector:Micro_SD_Card_Det J1
+L MCT_Labor_5529-rescue:Micro_SD_Card_Det-Connector J1
 U 1 1 5EF780A1
 P 3450 1700
@@
 $EndComp
 $Comp
-L power:GND #PWR0131
+L MCT_Labor_5529-rescue:GND-power #PWR0131
 U 1 1 5EF85C1B
 P 3950 4100
@@
 	5500 1950 5500 4000
 $Comp
-L power:+3.3V #PWR0132
+L MCT_Labor_5529-rescue:+3.3V-power #PWR0132
 U 1 1 5EF99555
 P 6150 900
@@
 	6150 900  6150 1050
 $Comp
-L power:GND #PWR0133
+L MCT_Labor_5529-rescue:GND-power #PWR0133
 U 1 1 5EF9A52E
 P 6150 2550
@@
 $EndComp
 $Comp
-L power:GND #PWR0134
+L MCT_Labor_5529-rescue:GND-power #PWR0134
 U 1 1 5EF9A881
 P 6850 2550
@@
 $EndComp
 $Comp
-L power:+3.3V #PWR0135
+L MCT_Labor_5529-rescue:+3.3V-power #PWR0135
 U 1 1 5EF9ABE8
 P 6850 900
@@
 $EndComp
 $Comp
-L Device:C_Small C6
+L MCT_Labor_5529-rescue:C_Small-Device C6
 U 1 1 5EF9BD19
 P 6850 1650
@@
 	6150 2550 6150 2250
 $Comp
-L Device:R_Small R17
+L MCT_Labor_5529-rescue:R_Small-Device R17
 U 1 1 5F2E010A
 P 4300 3400
@@
 $EndComp
 $Comp
-L power:GND #PWR0136
+L MCT_Labor_5529-rescue:GND-power #PWR0136
 U 1 1 5F2E0E1E
 P 4300 4100
@@
 	4300 900  3950 900
 $Comp
-L 74xx:74HCT595 U6
+L MCT_Labor_5529-rescue:74HCT595-74xx U6
 U 1 1 5F3370D8
 P 8400 1700
+AR Path="/5F3370D8" Ref="U6"  Part="1"
+AR Path="/5EF44B02/5F3370D8" Ref="U6"  Part="1"
 F 0 "U6" H 8150 2250 50  0000 C CNN
 F 1 "74HCT595" H 8650 2250 50  0000 C CNN
@@
 $EndComp
 $Comp
-L power:GND #PWR0137
+L MCT_Labor_5529-rescue:GND-power #PWR0137
 U 1 1 5F33E16C
 P 9850 2550
@@
 $EndComp
 $Comp
-L power:+3.3V #PWR0138
+L MCT_Labor_5529-rescue:+3.3V-power #PWR0138
 U 1 1 5F33E172
 P 9850 900
@@
 $EndComp
 $Comp
-L Device:C_Small C8
+L MCT_Labor_5529-rescue:C_Small-Device C8
 U 1 1 5F33E178
 P 9850 1650
@@
 	9850 1750 9850 2550
 $Comp
-L power:+3.3V #PWR0139
+L MCT_Labor_5529-rescue:+3.3V-power #PWR0139
 U 1 1 5F33FF8C
 P 8400 900
@@
 	8400 900  8400 1100
 $Comp
-L power:GND #PWR0140
+L MCT_Labor_5529-rescue:GND-power #PWR0140
 U 1 1 5F342A21
 P 8400 2550
@@
 	7500 1800 8000 1800
 $Comp
-L Device:R_Small R19
+L MCT_Labor_5529-rescue:R_Small-Device R19
 U 1 1 5F34F536
 P 7900 2350
@@
 $EndComp
 $Comp
-L Device:C_Small C7
+L MCT_Labor_5529-rescue:C_Small-Device C7
 U 1 1 5F350180
 P 7700 2350
@@
 	7900 1900 7900 2250
 $Comp
-L power:GND #PWR0141
+L MCT_Labor_5529-rescue:GND-power #PWR0141
 U 1 1 5F35E09E
 P 7900 2550
@@
 $EndComp
 $Comp
-L power:GND #PWR0142
+L MCT_Labor_5529-rescue:GND-power #PWR0142
 U 1 1 5F35E4CA
 P 7700 2550
@@
 	7900 2450 7900 2550
 $Comp
-L Device:R_Small R18
+L MCT_Labor_5529-rescue:R_Small-Device R18
 U 1 1 5F34FB26
 P 7700 1100
@@
 $EndComp
 $Comp
-L power:+3.3V #PWR0143
+L MCT_Labor_5529-rescue:+3.3V-power #PWR0143
 U 1 1 5F363992
 P 7700 900
@@
 	7700 900  7700 1000
 $Comp
-L Device:LED_Small D2
+L MCT_Labor_5529-rescue:LED_Small-Device D2
 U 1 1 5F37CF38
 P 8900 1300
@@
 $EndComp
 $Comp
-L Device:R_Small R20
+L MCT_Labor_5529-rescue:R_Small-Device R20
 U 1 1 5F392D5A
 P 9350 1300
@@
 	9000 1300 9250 1300
 $Comp
-L Device:LED_Small D3
+L MCT_Labor_5529-rescue:LED_Small-Device D3
 U 1 1 5F3976BD
 P 8900 1400
@@
 $EndComp
 $Comp
-L Device:R_Small R21
+L MCT_Labor_5529-rescue:R_Small-Device R21
 U 1 1 5F3976C3
 P 9350 1400
@@
 	9000 1400 9250 1400
 $Comp
-L Device:LED_Small D4
+L MCT_Labor_5529-rescue:LED_Small-Device D4
 U 1 1 5F398E51
 P 8900 1500
@@
 $EndComp
 $Comp
-L Device:R_Small R22
+L MCT_Labor_5529-rescue:R_Small-Device R22
 U 1 1 5F398E57
 P 9350 1500
@@
 	9000 1500 9250 1500
 $Comp
-L Device:LED_Small D5
+L MCT_Labor_5529-rescue:LED_Small-Device D5
 U 1 1 5F39A666
 P 8900 1600
@@
 $EndComp
 $Comp
-L Device:R_Small R23
+L MCT_Labor_5529-rescue:R_Small-Device R23
 U 1 1 5F39A66C
 P 9350 1600
@@
 	9000 1600 9250 1600
 $Comp
-L Device:LED_Small D6
+L MCT_Labor_5529-rescue:LED_Small-Device D6
 U 1 1 5F39BEEF
 P 8900 1700
@@
 $EndComp
 $Comp
-L Device:R_Small R24
+L MCT_Labor_5529-rescue:R_Small-Device R24
 U 1 1 5F39BEF5
 P 9350 1700
@@
 	9000 1700 9250 1700
 $Comp
-L Device:LED_Small D7
+L MCT_Labor_5529-rescue:LED_Small-Device D7
 U 1 1 5F39D815
 P 8900 1800
@@
 $EndComp
 $Comp
-L Device:R_Small R25
+L MCT_Labor_5529-rescue:R_Small-Device R25
 U 1 1 5F39D81B
 P 9350 1800
@@
 	9000 1800 9250 1800
 $Comp
-L Device:LED_Small D8
+L MCT_Labor_5529-rescue:LED_Small-Device D8
 U 1 1 5F39F1EB
 P 8900 1900
@@
 $EndComp
 $Comp
-L Device:R_Small R26
+L MCT_Labor_5529-rescue:R_Small-Device R26
 U 1 1 5F39F1F1
 P 9350 1900
@@
 	9000 1900 9250 1900
 $Comp
-L Device:LED_Small D9
+L MCT_Labor_5529-rescue:LED_Small-Device D9
 U 1 1 5F3A0BEC
 P 8900 2000
@@
 $EndComp
 $Comp
-L Device:R_Small R27
+L MCT_Labor_5529-rescue:R_Small-Device R27
 U 1 1 5F3A0BF2
 P 9350 2000
@@
 	9000 2000 9250 2000
 $Comp
-L power:GND #PWR0144
+L MCT_Labor_5529-rescue:GND-power #PWR0144
 U 1 1 5F3A961C
 P 9650 2550
@@
 	2800 5350 7500 5350
 $Comp
-L Connector_Generic:Conn_02x05_Odd_Even J2
+L MCT_Labor_5529-rescue:Conn_02x05_Odd_Even-Connector_Generic J2
 U 1 1 5F3F06A3
 P 4250 5650
@@
 	5200 5650 5200 3000
 $Comp
-L power:GND #PWR0145
+L MCT_Labor_5529-rescue:GND-power #PWR0145
 U 1 1 5F4209BC
 P 5400 6050
@@
 $EndComp
 $Comp
-L power:+3.3V #PWR0146
+L MCT_Labor_5529-rescue:+3.3V-power #PWR0146
 U 1 1 5F420E46
 P 5400 5150
@@
 	5400 5750 5400 6050
 $Comp
-L Device:C_Small C5
+L MCT_Labor_5529-rescue:C_Small-Device C5
 U 1 1 5F43BA8E
 P 5400 5650

Commit message: Aktuell gefertigte Variante
Parts:
- R20, R21, R22, R23, R24, R25, R26, R27: value 220 -> 1k
Changed lines of the file:
@@
 P 9350 1300
 F 0 "R20" V 9300 1200 50  0000 R CNN
-F 1 "220" V 9300 1400 50  0000 L CNN
+F 1 "1k" V 9300 1400 50  0000 L CNN
 F 2 "Resistor_SMD:R_0603_1608Metric_Pad1.05x0.95mm_HandSolder" H 9350 1300 50  0001 C CNN
 F 3 "~" H 9350 1300 50  0001 C CNN
@@
 P 9350 1400
 F 0 "R21" V 9300 1300 50  0000 R CNN
-F 1 "220" V 9300 1500 50  0000 L CNN
+F 1 "1k" V 9300 1500 50  0000 L CNN
 F 2 "Resistor_SMD:R_0603_1608Metric_Pad1.05x0.95mm_HandSolder" H 9350 1400 50  0001 C CNN
 F 3 "~" H 9350 1400 50  0001 C CNN
@@
 P 9350 1500
 F 0 "R22" V 9300 1400 50  0000 R CNN
-F 1 "220" V 9300 1600 50  0000 L CNN
+F 1 "1k" V 9300 1600 50  0000 L CNN
 F 2 "Resistor_SMD:R_0603_1608Metric_Pad1.05x0.95mm_HandSolder" H 9350 1500 50  0001 C CNN
 F 3 "~" H 9350 1500 50  0001 C CNN
@@
 P 9350 1600
 F 0 "R23" V 9300 1500 50  0000 R CNN
-F 1 "220" V 9300 1700 50  0000 L CNN
+F 1 "1k" V 9300 1700 50  0000 L CNN
 F 2 "Resistor_SMD:R_0603_1608Metric_Pad1.05x0.95mm_HandSolder" H 9350 1600 50  0001 C CNN
 F 3 "~" H 9350 1600 50  0001 C CNN
@@
 P 9350 1700
 F 0 "R24" V 9300 1600 50  0000 R CNN
-F 1 "220" V 9300 1800 50  0000 L CNN
+F 1 "1k" V 9300 1800 50  0000 L CNN
 F 2 "Resistor_SMD:R_0603_1608Metric_Pad1.05x0.95mm_HandSolder" H 9350 1700 50  0001 C CNN
 F 3 "~" H 9350 1700 50  0001 C CNN
@@
 P 9350 1800
 F 0 "R25" V 9300 1700 50  0000 R CNN
-F 1 "220" V 9300 1900 50  0000 L CNN
+F 1 "1k" V 9300 1900 50  0000 L CNN
 F 2 "Resistor_SMD:R_0603_1608Metric_Pad1.05x0.95mm_HandSolder" H 9350 1800 50  0001 C CNN
 F 3 "~" H 9350 1800 50  0001 C CNN
@@
 P 9350 1900
 F 0 "R26" V 9300 1800 50  0000 R CNN
-F 1 "220" V 9300 2000 50  0000 L CNN
+F 1 "1k" V 9300 2000 50  0000 L CNN
 F 2 "Resistor_SMD:R_0603_1608Metric_Pad1.05x0.95mm_HandSolder" H 9350 1900 50  0001 C CNN
 F 3 "~" H 9350 1900 50  0001 C CNN
@@
 P 9350 2000
 F 0 "R27" V 9300 1900 50  0000 R CNN
-F 1 "220" V 9300 2100 50  0000 L CNN
+F 1 "1k" V 9300 2100 50  0000 L CNN
 F 2 "Resistor_SMD:R_0603_1608Metric_Pad1.05x0.95mm_HandSolder" H 9350 2000 50  0001 C CNN
 F 3 "~" H 9350 2000 50  0001 C CNN
